Commit message: added virtual camera for recording in gazebo

File: urdf/left_arm.xacro (robot description, xacro)
@@ -20,4 +20,5 @@
     <xacro:property name="axel_offset" value="0.05" /> <!-- Space btw top of beam and the each joint -->
     <xacro:property name="damping" value="0.7" /> <!-- damping factor -->
+    <xacro:property name="camera_link" value="0.05" /> <!-- Size of square 'camera' box -->
     <!-- Import all Gazebo-customization elements, including Gazebo colors -->
     <xacro:include filename="$(find raven_2arm)/urdf/raven_2arm.gazebo" />

File: urdf/raven_2arm.xacro (robot description, xacro)
@@ -77,4 +77,25 @@
         </inertial>
     </link>
+    <!-- Camera -->
+    <link name="camera_link">
+        <collision>
+          <origin xyz="0 0 0" rpy="0 0 0"/>
+          <geometry>
+        <box size="${camera_link} ${camera_link} ${camera_link}"/>
+          </geometry>
+        </collision>
+        <visual>
+          <origin xyz="0 0 0" rpy="0 0 0"/>
+          <geometry>
+        <box size="${camera_link} ${camera_link} ${camera_link}"/>
+          </geometry>
+          <material name="red"/>
+        </visual>
+        <inertial>
+          <mass value="1e-5" />
+          <origin xyz="0 0 0" rpy="0 0 0"/>
+          <inertia ixx="1e-6" ixy="0" ixz="0" iyy="1e-6" iyz="0" izz="1e-6" />
+        </inertial>
+      </link>
     <!-- LEFT ARM JOINTS -->
     <joint name="camera_L" type="fixed">
@@ -85,4 +106,11 @@
         <child link="base_link_L"/>
     </joint>
+    <!-- Added by Samin for virtual Camera -->
+    <joint name="camera_joint" type="fixed">
+        <axis xyz="0 0 0" />
+        <origin xyz="-0.265 0.200 0.1" rpy="0 0 -1.57"/>
+        <parent link="world"/>
+        <child link="camera_link"/>
+      </joint>
     <link name="link1_L">
         <visual>
