Commit message: change some pythysical parameters, like mass, inertia

File: urdf/raven_2arm.xacro (robot description, xacro)
@@ -19,5 +19,6 @@
     <xacro:property name="camera_link" value="0.05" /> <!-- Size of square 'camera' box -->
     <xacro:property name="axel_offset" value="0.05" /> <!-- Space btw top of beam and the each joint -->
-    <xacro:property name="damping" value="0.7" /> <!-- damping factor -->
+    <xacro:property name="damping" value="0.5" /> <!-- damping factor -->
+    <xacro:property name="friction" value="0.2" /> <!-- friction factor -->
     <!-- Import all Gazebo-customization elements, including Gazebo colors -->
     <xacro:include filename="$(find raven_2arm)/urdf/raven_2arm.gazebo" />
@@ -110,5 +111,5 @@
         <parent link="base_link_L"/>
         <child link="link1_L"/>
-        <dynamics damping="${damping}"/>
+        <dynamics damping="${damping}" friction="${friction}"/>
     </joint>
     <link name="link2_L">
@@ -137,5 +138,5 @@
         <parent link="link1_L"/>
         <child link="link2_L"/>
-        <dynamics damping="${damping}"/>
+        <dynamics damping="${damping}" friction="0.5"/>
     </joint>
     <link name="link3_L">
@@ -164,5 +165,5 @@
         <parent link="link2_L"/>
         <child link="link3_L"/>
-        <dynamics damping="${damping}"/>
+        <dynamics damping="${damping}" friction="${friction}"/>
     </joint>
     <link name="instrument_shaft_L">
@@ -191,5 +192,5 @@
         <parent link="link3_L"/>
         <child link="instrument_shaft_L"/>
-        <dynamics damping="${damping}"/>
+        <dynamics damping="${damping}" friction="${friction}"/>
     </joint>
     <link name="wrist_L">
@@ -218,5 +219,5 @@
         <parent link="instrument_shaft_L"/>
         <child link="wrist_L"/>
-        <dynamics damping="${damping}"/>
+        <dynamics damping="${damping}" friction="${friction}"/>
     </joint>
     <link name="grasper1_L">
@@ -308,5 +309,5 @@
         <parent link="world"/>
         <child link="base_link_R"/>
-        <dynamics damping="${damping}"/>
+        <dynamics damping="${damping}" friction="${friction}"/>
     </joint>
     <link name="link1_R">
@@ -339,5 +340,5 @@
         <parent link="base_link_R"/>
         <child link="link1_R"/>
-        <dynamics damping="${damping}"/>
+        <dynamics damping="${damping}" friction="${friction}"/>
     </joint>
     <link name="link2_R">
@@ -369,5 +370,5 @@
         <parent link="link1_R"/>
         <child link="link2_R"/>
-        <dynamics damping="${damping}"/>
+        <dynamics damping="${damping}" friction="${friction}"/>
     </joint>
     <link name="link3_R">
@@ -399,5 +400,5 @@
         <parent link="link2_R"/>
         <child link="link3_R"/>
-        <dynamics damping="${damping}"/>
+        <dynamics damping="${damping}" friction="${friction}"/>
     </joint>
     <link name="instrument_shaft_R">
@@ -429,5 +430,5 @@
         <parent link="link3_R"/>
         <child link="instrument_shaft_R"/>
-        <dynamics damping="${damping}"/>
+        <dynamics damping="${damping}" friction="${friction}"/>
     </joint>
     <link name="wrist_R">
@@ -459,5 +460,5 @@
         <parent link="instrument_shaft_R"/>
         <child link="wrist_R"/>
-        <dynamics damping="${damping}"/>
+        <dynamics damping="${damping}" friction="${friction}"/>
     </joint>
     <link name="grasper1_R">

File: urdf/raven_gazebo_6dof.urdf (robot description, URDF)
Before this commit: robot raven_2arm, 18 links, 17 joints
Links:
- removed link grasper2_L
- removed link grasper2_R
Joints:
- removed joint grasper_joint_2_L
- removed joint grasper_joint_2_R
